Commit message: fix(p3d): joint is fixed instead of revolute

File: simulation/ruvu_sensor_descriptions/urdf_xacro/generic_p3d_sensor.urdf.xacro (robot description, xacro)
@@ -4,6 +4,5 @@
     <xacro:macro name="generic_p3d_sensor_model" params="name parent *origin">
      <!-- use a zero limit revolute joint rather than fixed to prevent lumping -->
-      <joint name="${name}_joint" type="revolute">
-        <limit effort="0" lower="0" upper="0" velocity="0"/>
+      <joint name="${name}_joint" type="fixed">
         <xacro:insert_block name="origin" />
         <parent link="${parent}"/>

Commit message: Revert "fix(p3d): joint is fixed instead of revolute"
This reverts commit b29eab44311ada4018d9f374c331860aa4b91cda.

File: simulation/ruvu_sensor_descriptions/urdf_xacro/generic_p3d_sensor.urdf.xacro (robot description, xacro)
@@ -4,5 +4,6 @@
     <xacro:macro name="generic_p3d_sensor_model" params="name parent *origin">
      <!-- use a zero limit revolute joint rather than fixed to prevent lumping -->
-      <joint name="${name}_joint" type="fixed">
+      <joint name="${name}_joint" type="revolute">
+        <limit effort="0" lower="0" upper="0" velocity="0"/>
         <xacro:insert_block name="origin" />
         <parent link="${parent}"/>

Commit message: fix(p3d_sensor): 1cm block

File: simulation/ruvu_sensor_descriptions/urdf_xacro/generic_p3d_sensor.urdf.xacro (robot description, xacro)
@@ -12,18 +12,18 @@
       <link name="${name}">
         <inertial>
-          <mass value="0.270" />
+          <mass value="0.070" />
           <origin xyz="0 0 0" rpy="0 0 0" />
           <inertia ixx="2.632e-4" ixy="0" ixz="0" iyy="2.632e-4" iyz="0" izz="1.62e-4" />
         </inertial>
         <visual>
-          <origin xyz="0 0 -0.0115" rpy="0 0 0" />
+          <origin xyz="0 0 0.005" rpy="0 0 0" />
           <geometry>
-          <box size="0.058 0.058 0.087" />
+          <box size="0.01 0.01 0.01" />
         </geometry>
         </visual>
         <collision>
-          <origin xyz="0 0 -0.0115" rpy="0 0 0" />
+          <origin xyz="0 0 0.005" rpy="0 0 0" />
           <geometry>
-          <box size="0.058 0.058 0.087" />
+          <box size="0.01 0.01 0.01" />
         </geometry>
         </collision>
