Commit message: wip(rgb_led_plugin): Almost working model plugin

File: simulation/ruvu_gazebo_plugins/test/rgb_led_visual.urdf (robot description, URDF)
Before this commit: robot robot, 1 links, 0 joints
Links:
- removed link base_link
- added link led1; visual box size=0.1 0.1 0.1
- added link led2; visual box size=0.1 0.1 0.1
- added link led3; visual box size=0.1 0.1 0.1
- added link led4; visual box size=0.1 0.1 0.1
- added link led5; visual box size=0.1 0.1 0.1
- added link mount, mass 0.01; collision box size=3.0 1.0 1.0; visual box size=3.0 1.0 1.0
Joints:
- added joint led1_joint: type revolute, parent mount, child led1, origin xyz=-1.5 0 1.0 rpy=0 0 0, limit lower=0 upper=0 effort=0 velocity=0
- added joint led2_joint: type revolute, parent mount, child led2, origin xyz=-0.75 0 1.0 rpy=0 0 0, limit lower=0 upper=0 effort=0 velocity=0
- added joint led3_joint: type revolute, parent mount, child led3, origin xyz=0 0 1.0 rpy=0 0 0, limit lower=0 upper=0 effort=0 velocity=0
- added joint led4_joint: type revolute, parent mount, child led4, origin xyz=0.75 0 1.0 rpy=0 0 0, limit lower=0 upper=0 effort=0 velocity=0
- added joint led5_joint: type revolute, parent mount, child led5, origin xyz=1.5 0 1.0 rpy=0 0 0, limit lower=0 upper=0 effort=0 velocity=0

Commit message: wip(rgb_plugin): SDF is working

File: simulation/ruvu_gazebo_plugins/test/rgb_led_visual.urdf (robot description, URDF)
Before this commit: robot robot, 6 links, 5 joints
Joints:
- joint led1_joint: limit lower=0 upper=0 effort=0 velocity=0 -> (none); type revolute -> fixed
- joint led2_joint: limit lower=0 upper=0 effort=0 velocity=0 -> (none); type revolute -> fixed
- joint led3_joint: limit lower=0 upper=0 effort=0 velocity=0 -> (none); type revolute -> fixed
- joint led4_joint: limit lower=0 upper=0 effort=0 velocity=0 -> (none); type revolute -> fixed
- joint led5_joint: limit lower=0 upper=0 effort=0 velocity=0 -> (none); type revolute -> fixed
